Commit message: Improvements on simulation, it now launches but x axis simulation is bugged

File: install/eye_on_you/share/eye_on_you/robot.urdf (robot description, URDF)
Before this commit: robot robot, 4 links, 3 joints
Joints:
- joint base_home_joint: axis 0 0 1 -> 0 1 0; origin xyz=0 0 0.024 -> xyz=1.47 31.7 -40.5
- joint home_arm_joint: axis 0 0 1 -> 1 0 0; origin xyz=0.014 0 0.029 rpy=1.5707 -1.5707 0 -> xyz=-12 57.6 -58.9 rpy=0 0 0

Commit message: Fixed arm on simulation

File: install/eye_on_you/share/eye_on_you/robot.urdf (robot description, URDF)
Before this commit: robot robot, 4 links, 3 joints
Joints:
- joint home_arm_joint: origin xyz=-12 57.6 -58.9 rpy=0 0 0 -> xyz=-13.5 26 -18.5
